File: diy-ham-radio-dds/diy-ham-radio-dds.kicad_pcb (KiCad board)
At the start: 2 copper layers, 150 x 50 mm, 63 parts, among them J1 I2C, J2 ICSP, J3 VCC, J4 NPN OUT, J5 , J6 UART_PROG, Q1 S0805, Q2 S0805, Q3 S0805, Q4 S0805, Q5 S0805, Q6 S0805, Q7 S0805, Q8 S0805, SW1 SW_Push, SW2 SW_Push, SW3 SW_Push, SW4 SW_Push, SW5 Rotary_Encoder_Switch, U1 ATmega328-AU, U2 74LS08, U3 L7805, U4 74HC595, Y1 16MHz

Commit message: Drawing in progress
Parts:
- removed the R5 at (184.4, 77.0)
- removed the R6 at (197.7, 76.2)
- added R10: 1k, Resistor_SMD:R_0402_1005Metric, B.Cu at (264.4, 147.1)
- added R11: 0R, Resistor_SMD:R_0805_2012Metric, B.Cu at (201.8, 54.3)
- C10, C11, C12, C13, C2, C3, C4, C6, C7, C8, C9, D1, D2, J3, J4, J5, J6, Q1, Q2, Q3, Q4, Q5, Q6, Q7, Q8, R1, R2, R3, U2, U3, U4, Y1: moved to B.Cu
- J1: renamed from J2; moved to B.Cu
- J2: renamed from J1; moved to B.Cu
- R12: renamed from R10; moved to B.Cu
- R13: renamed from R11; moved to B.Cu
- R14: renamed from R12; moved to B.Cu
- R15: renamed from R13; moved to B.Cu
- R16: renamed from R14; moved to B.Cu
- R17: renamed from R15; moved to B.Cu
- R18: renamed from R16; moved to B.Cu
- R19: renamed from R17; moved to B.Cu
- R20: renamed from R18; moved to B.Cu
- R4: renamed from R19; moved to B.Cu
- R5: renamed from R20; moved to B.Cu
- R6: renamed from R4; moved to B.Cu
- R7, R8: footprint Resistor_SMD:R_Array_Convex_4x0402 -> Resistor_SMD:R_0402_1005Metric; moved to B.Cu
- R9: value 0R -> 1k; footprint Resistor_SMD:R_0805_2012Metric -> Resistor_SMD:R_0402_1005Metric; moved to B.Cu
- moved J4 136.4 mm to (276.0, 135.0), turned to 270 degrees
- moved Y1 122.9 mm to (265.4, 142.1), turned to 270 degrees
- moved J5 112.9 mm to (188.8, 157.1)
- moved Q7 112.3 mm to (270.3, 149.1), turned to 270 degrees
- moved Q8 109.1 mm to (270.3, 152.7), turned to 270 degrees
- moved R7 105.6 mm to (265.4, 135.6), turned to 270 degrees
- moved Q3 105.3 mm to (270.3, 134.7), turned to 270 degrees
- moved R16 105.2 mm to (266.4, 150.7), turned to 180 degrees
- moved U2 105.0 mm to (257.6, 150.6), turned to 90 degrees
- moved Q5 103.6 mm to (270.3, 141.9), turned to 270 degrees
- moved Q6 102.6 mm to (270.3, 145.5), turned to 270 degrees
- moved R17 101.0 mm to (265.9, 152.0), turned to 180 degrees
- moved Q1 101.0 mm to (277.2, 129.5), turned to 270 degrees
- moved Q2 99.9 mm to (277.2, 125.8), turned to 270 degrees
- moved R15 99.2 mm to (266.8, 147.1), turned to 270 degrees
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Connections:
- R7 pad 1: Net-(Q3-Pad1) -> Net-(Q1-Pad1)
- R7 pad 2: Q3_NPN -> Q1_NPN
- R8 pad 1: Net-(Q4-Pad1) -> Net-(Q2-Pad1)
- R8 pad 2: Q4_NPN -> Q2_NPN
- R9 pad 1: VCC -> Net-(Q3-Pad1)
- R9 pad 2: POT1_A -> Q3_NPN
- U1 pad 23: DISP_D4 -> SHIFT_ENABLE
- U1 pad 24: SHIFT_ENABLE -> DISP_D4
- Y1 pad 2: Net-(C8-Pad2) -> GND
- Y1 pad 3: (no net) -> Net-(C8-Pad2)
- Y1 pad 4: (no net) -> GND
Routing:
- net SHIFT_ENABLE: track 0.00 -> 32.8 mm, vias 0 -> 2
- net Q2_NPN: track 0.00 -> 24.8 mm, vias 0 -> 1
- net Q1_NPN: track 0.00 -> 24.3 mm, vias 0 -> 1
- net Q3_NPN: track 0.00 -> 23.7 mm, vias 0 -> 1
- net Net-(Q2-Pad1): track 0.00 -> 22.0 mm
- net Net-(Q1-Pad1): track 0.00 -> 18.5 mm
- net Q2: track 0.00 -> 15.1 mm
- net Net-(Q4-Pad1): track 0.00 -> 13.4 mm
- net Q6_NPN: track 0.00 -> 12.1 mm, vias 0 -> 1
- net Q4_NPN: track 0.00 -> 12.1 mm, vias 0 -> 1
- net Q5_NPN: track 0.00 -> 11.9 mm, vias 0 -> 1
- net DISP_D6\SHIFT_LATCH: track 135.9 -> 147.2 mm
- net Q7_NPN: track 0.00 -> 10.3 mm, vias 0 -> 1
- net SHIFT_DATA: track 0.00 -> 10.3 mm, vias 0 -> 1
- net Q3: track 0.00 -> 9.78 mm
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
Commit message: Drawing in progress
Parts:
- C1, C10, C11, C13, C5, C6, C9, J1, J2, J3, J5, J6, R11, R12, R13, R18, R19, R20, U3: moved to F.Cu
- R2: footprint Resistor_SMD:R_0402_1005Metric_Pad0.72x0.64mm_HandSolder -> Resistor_SMD:R_0402_1005Metric; moved to F.Cu
- R3: footprint Resistor_SMD:R_01005_0402Metric -> Resistor_SMD:R_0402_1005Metric; moved to F.Cu
- R5: footprint Resistor_SMD:R_0402_1005Metric_Pad0.72x0.64mm_HandSolder -> Resistor_SMD:R_0402_1005Metric
- R6: footprint Resistor_SMD:R_01005_0402Metric_Pad0.57x0.30mm_HandSolder -> Resistor_SMD:R_0402_1005Metric; moved to F.Cu
- moved R6 160.2 mm to (237.0, 190.6)
- moved R3 158.2 mm to (258.8, 176.7)
- moved R2 156.4 mm to (226.6, 194.0)
- moved R20 153.4 mm to (254.9, 183.6)
- moved J3 152.6 mm to (245.6, 183.4)
- moved C13 148.1 mm to (254.1, 188.0)
- moved U3 147.8 mm to (243.0, 179.8)
- moved R11 145.2 mm to (246.7, 192.3)
- moved C11 143.3 mm to (254.1, 186.0)
- moved J2 142.8 mm to (250.0, 183.4)
- moved J1 141.1 mm to (233.0, 191.3)
- moved C9 140.5 mm to (250.4, 190.9)
- moved RV1 138.7 mm to (226.7, 180.3)
- moved R12 136.2 mm to (246.2, 189.4)
- moved C6 132.8 mm to (258.5, 184.1)
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Connections:
- J5 pad 1: VCC -> POT2_A
- J5 pad 10: ALARM -> Net-(J5-Pad10)
- J5 pad 2: GND -> POT2_B
- J5 pad 3: POT1_A -> POT2_C
- J5 pad 4: POT1_B -> POT1_A
- J5 pad 5: POT1_C -> POT1_B
- J5 pad 6: POT2_A -> POT1_C
- J5 pad 7: POT2_B -> PTT
- J5 pad 8: POT2_C -> ALARM
- J5 pad 9: PTT -> Net-(J5-Pad9)
Routing:
- net DISP_D4: track 167.3 -> 328.1 mm
- net VCC: track 21.7 -> 128.6 mm
- net POT_2: track 0.00 -> 42.4 mm
- net POT_1: track 0.00 -> 39.0 mm
- net ALARM_IN: track 0.00 -> 38.1 mm
- net Q7_NPN: track 10.3 -> 48.2 mm, vias 1 -> 2
- net Q8_NPN: track 5.92 -> 43.0 mm, vias 1 -> 2
- net Q5_NPN: track 11.9 -> 47.6 mm, vias 1 -> 2
- net Q4_NPN: track 12.1 -> 46.5 mm
- net Q2_NPN: track 24.8 -> 57.6 mm, vias 1 -> 2
- net Q3_NPN: track 23.7 -> 55.4 mm
- net RST: track 0.00 -> 31.7 mm
- net RX: track 0.00 -> 31.0 mm
- net TX: track 0.00 -> 30.2 mm
- net PTT_IN: track 0.86 -> 31.1 mm
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- added copper zone on B.Cu, net GND
- added copper zone on F.Cu, net GND
